File: keyboard.kicad_pcb (KiCad board)
At the start: 2 copper layers, 88 parts, among them SW1 SW_PUSH, SW10 SW_PUSH, SW11 SW_PUSH, SW12 SW_PUSH, SW13 SW_PUSH, SW14 SW_PUSH, SW15 SW_PUSH, SW16 SW_PUSH, SW17 SW_PUSH, SW18 SW_PUSH, SW19 SW_PUSH, SW2 SW_PUSH, SW20 SW_PUSH, SW21 SW_PUSH, SW22 SW_PUSH, SW23 SW_PUSH, SW24 SW_PUSH, SW25 SW_PUSH, SW26 SW_PUSH, SW27 SW_PUSH, SW28 SW_PUSH, SW29 SW_PUSH, SW3 SW_PUSH, SW30 SW_PUSH, SW31 SW_PUSH, SW32 SW_PUSH, SW33 SW_PUSH, SW34 SW_PUSH, SW35 SW_PUSH, SW36 SW_PUSH, SW37 SW_PUSH, SW38 SW_PUSH, SW39 SW_PUSH, SW4 SW_PUSH, SW40 SW_PUSH, SW41 SW_PUSH, SW42 SW_PUSH, SW43 SW_PUSH, SW5 SW_PUSH, SW6 SW_PUSH, SW7 SW_PUSH, SW8 SW_PUSH, SW9 SW_PUSH, U1 Pico

Commit message: :construction:
Parts:
- D1, D10, D11, D12, D13, D14, D15, D16, D17, D18, D19, D2, D20, D21, D22, D23, D24, D25, D26, D27, D28, D29, D3, D30, D31, D32, D33, D34, D35, D36, D37, D38, D39, D4, D40, D41, D42, D43, D5, D6, D7, D8, D9: footprint kbd:D3_SMD_v2 -> Diode_SMD:D_SOD-123; moved to B.Cu
- SW_RESET1: moved to B.Cu
- moved SW_RESET1 201.4 mm to (349.0, 67.0), turned to -90 degrees
- moved D35 158.6 mm to (333.4, 88.1), turned to -90 degrees
- moved D11 153.1 mm to (304.8, 50.0), turned to -90 degrees
- moved D12 142.4 mm to (333.4, 50.0), turned to -90 degrees
- moved D10 142.3 mm to (285.8, 50.0), turned to -90 degrees
- moved D9 136.2 mm to (266.7, 50.0), turned to -90 degrees
- moved D1 133.5 mm to (114.3, 50.0), turned to -90 degrees
- moved D24 133.4 mm to (340.5, 69.1), turned to -90 degrees
- moved D36 130.0 mm to (121.4, 107.2), turned to -90 degrees
- moved D42 128.6 mm to (311.9, 107.2), turned to -90 degrees
- moved D41 128.4 mm to (288.1, 107.2), turned to -90 degrees
- moved D43 125.4 mm to (335.8, 107.2), turned to -90 degrees
- moved D3 122.4 mm to (152.4, 50.0), turned to -90 degrees
- moved D14 121.8 mm to (138.1, 69.1), turned to -90 degrees
- moved D8 120.3 mm to (247.7, 50.0), turned to -90 degrees
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Connections:
- U1 pad 11: col2 -> row7
- U1 pad 12: col3 -> row6
- U1 pad 21: row6 -> col2
- U1 pad 22: row7 -> col3
Routing:
- net col3: track 0.00 -> 350.3 mm
- net col1: track 0.00 -> 319.6 mm
- net col0: track 0.00 -> 317.7 mm
- net col2: track 0.00 -> 307.9 mm
- net Net-(D35-Pad2): track 0.00 -> 12.4 mm
- net Net-(D36-Pad2): track 0.00 -> 11.9 mm
- net Net-(D13-Pad2): track 0.00 -> 11.6 mm
- net Net-(D37-Pad2): track 0.00 -> 11.5 mm
- net Net-(D12-Pad2): track 0.00 -> 11.4 mm
- net Net-(D32-Pad2): track 0.00 -> 11.4 mm
- net Net-(D39-Pad2): track 0.00 -> 11.3 mm
- net Net-(D30-Pad2): track 0.00 -> 11.3 mm
- net Net-(D8-Pad2): track 0.00 -> 11.3 mm
- net Net-(D28-Pad2): track 0.00 -> 11.3 mm
- net Net-(D43-Pad2): track 0.00 -> 11.3 mm
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Other:
- board outline added: 269.5 x 79.5 mm

Commit message: :construction:
Parts:
- added D44: D, Diode_SMD:D_SOD-123, F.Cu at (110.6, 48.7)
- added D45: D, Diode_SMD:D_SOD-123, F.Cu at (70.3, 89.1)
- added D46: D, Diode_SMD:D_SOD-123, F.Cu at (116.3, 48.7)
- added D47: D, Diode_SMD:D_SOD-123, F.Cu at (76.0, 89.1)
- added D48: D, Diode_SMD:D_SOD-123, F.Cu at (217.7, 65.4)
- added D49: D, Diode_SMD:D_SOD-123, F.Cu at (223.5, 65.4)
- added SW44: SW_PUSH, mikamo3:CherryMX_Hotswap_1u, F.Cu at (258.2, 103.5)
- added SW45: SW_PUSH, mikamo3:CherryMX_Hotswap_1u, F.Cu at (277.3, 103.5)
- added SW46: SW_PUSH, mikamo3:CherryMX_Hotswap_1u, F.Cu at (296.3, 103.5)
- added SW47: SW_PUSH, mikamo3:CherryMX_Hotswap_1u, F.Cu at (315.4, 103.5)
- added SW48: RotaryEncoder_Switch, Rotary_Encoder:RotaryEncoder_Alps_EC12E-Switch_Vertical_H20mm, F.Cu at (235.4, 53.4)
- added SW49: RotaryEncoder_Switch, Rotary_Encoder:RotaryEncoder_Alps_EC12E-Switch_Vertical_H20mm, F.Cu at (216.9, 53.4)
- moved D25 80.1 mm to (113.0, 167.8)
- moved D26 80.1 mm to (139.2, 167.8)
- moved D27 80.1 mm to (158.2, 167.8)
- moved D28 80.1 mm to (177.3, 167.8)
- moved D29 80.1 mm to (196.3, 167.8)
- moved D30 80.1 mm to (215.4, 167.8)
- moved D31 80.1 mm to (234.4, 167.8)
- moved D32 80.1 mm to (253.5, 167.8)
- moved D33 80.1 mm to (272.5, 167.8)
- moved D34 80.1 mm to (291.6, 167.8)
- moved D35 80.1 mm to (324.9, 167.8)
- moved SW1 80.1 mm to (96.3, 127.3)
- moved SW10 80.1 mm to (267.8, 127.3)
- moved SW11 80.1 mm to (286.8, 127.3)
- moved SW12 80.1 mm to (315.4, 127.3)
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Connections:
- U1 pad 29: unconnected-(U1-Pad29) -> enc_0_a
- U1 pad 31: unconnected-(U1-Pad31) -> enc_0_b
- U1 pad 32: unconnected-(U1-Pad32) -> enc_1_a
- U1 pad 34: unconnected-(U1-Pad34) -> enc_1_b
- U1 pad 7: unconnected-(U1-Pad7) -> col4

Commit message: :construction:
Parts:
- removed D44, D45, D46, D47, D48, D49: D, Diode_SMD:D_SOD-123
- removed SW44, SW45, SW46, SW47: SW_PUSH, mikamo3:CherryMX_Hotswap_1u
- removed SW48, SW49: RotaryEncoder_Switch, Rotary_Encoder:RotaryEncoder_Alps_EC12E-Switch_Vertical_H20mm
- added LED1: YS-SK6812MINI-E, mikamo3:YS-SK6812MINI-E, F.Cu at (86.8, 129.7)
- added LED10: YS-SK6812MINI-E, mikamo3:YS-SK6812MINI-E, F.Cu at (205.8, 189.2)
- added LED11: YS-SK6812MINI-E, mikamo3:YS-SK6812MINI-E, F.Cu at (163.0, 189.2)
- added LED12: YS-SK6812MINI-E, mikamo3:YS-SK6812MINI-E, F.Cu at (115.4, 189.2)
- added LED13: YS-SK6812MINI-E, mikamo3:YS-SK6812MINI-E, F.Cu at (86.8, 170.2)
- added LED2: YS-SK6812MINI-E, mikamo3:YS-SK6812MINI-E, F.Cu at (105.8, 117.8)
- added LED3: YS-SK6812MINI-E, mikamo3:YS-SK6812MINI-E, F.Cu at (163.0, 117.8)
- added LED4: YS-SK6812MINI-E, mikamo3:YS-SK6812MINI-E, F.Cu at (239.2, 117.8)
- added LED5: YS-SK6812MINI-E, mikamo3:YS-SK6812MINI-E, F.Cu at (296.3, 117.8)
- added LED6: YS-SK6812MINI-E, mikamo3:YS-SK6812MINI-E, F.Cu at (334.4, 124.9)
- added LED7: YS-SK6812MINI-E, mikamo3:YS-SK6812MINI-E, F.Cu at (334.4, 170.2)
- added LED8: YS-SK6812MINI-E, mikamo3:YS-SK6812MINI-E, F.Cu at (305.9, 189.2)
- added LED9: YS-SK6812MINI-E, mikamo3:YS-SK6812MINI-E, F.Cu at (258.2, 189.2)
- moved U1 43.9 mm to (99.8, 146.0)
- moved SW_RESET1 27.7 mm to (365.4, 134.5)
- moved D36 4.76 mm to (113.0, 182.1), turned to 90 degrees
- moved D37 4.76 mm to (136.8, 182.1), turned to 90 degrees
- moved D38 4.76 mm to (160.6, 182.1), turned to 90 degrees
- moved D39 4.76 mm to (193.9, 182.1), turned to 90 degrees
- moved D40 4.76 mm to (241.6, 182.1), turned to 90 degrees
- moved D41 4.76 mm to (279.7, 182.1), turned to 90 degrees
- moved D42 4.76 mm to (303.5, 182.1), turned to 90 degrees
- moved D43 4.76 mm to (327.3, 182.1), turned to 90 degrees
- moved D35 2.38 mm to (322.5, 167.8), turned to 90 degrees
- turned D1 to 90 degrees
- turned D10 to 90 degrees
- turned D11 to 90 degrees
- turned D12 to 90 degrees
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Connections:
- SW40 pad 1: row4 -> row6
- SW41 pad 1: row5 -> row8
- SW42 pad 1: row6 -> row9
- SW43 pad 1: row7 -> row10
- U1 pad 1: unconnected-(U1-Pad1) -> led
- U1 pad 29: enc_0_a -> unconnected-(U1-Pad29)
- U1 pad 31: enc_0_b -> unconnected-(U1-Pad31)
- U1 pad 32: enc_1_a -> unconnected-(U1-Pad32)
- U1 pad 34: enc_1_b -> unconnected-(U1-Pad34)
- U1 pad 7: col4 -> unconnected-(U1-Pad7)
Routing:
- net VCC: track 0.00 -> 672.0 mm
- net col3: track 350.3 -> 249.7 mm
- net row10: track 0.00 -> 88.7 mm, vias 0 -> 4
- net row3: track 0.00 -> 86.6 mm, vias 0 -> 4
- net row9: track 0.00 -> 81.7 mm, vias 0 -> 4
- net row6: track 0.00 -> 78.1 mm, vias 0 -> 4
- net row8: track 0.00 -> 78.1 mm, vias 0 -> 4
- net row2: track 0.00 -> 75.6 mm, vias 0 -> 4
- net Net-(LED3-Pad2): track 0.00 -> 74.6 mm
- net col2: track 307.9 -> 245.7 mm
- net col0: track 317.7 -> 259.1 mm
- net Net-(LED2-Pad2): track 0.00 -> 55.3 mm
- net row7: track 0.00 -> 52.9 mm, vias 0 -> 3
- net row5: track 0.00 -> 52.9 mm, vias 0 -> 3
- net row4: track 0.00 -> 52.9 mm, vias 0 -> 3
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Other:
- board size 269.5 x 79.5 mm -> 277.7 x 90.2 mm

Commit message: :construction:
Parts:
- removed SW_RESET1: SW_Push, mikamo3:TactSwitch
Connections:
- U1 pad 10: col1 -> unconnected-(U1-Pad10)
- U1 pad 11: row7 -> col0
- U1 pad 12: row6 -> col1
- U1 pad 14: row0 -> row11
- U1 pad 15: row1 -> row6
- U1 pad 16: row2 -> row5
- U1 pad 17: row3 -> row4
- U1 pad 19: row4 -> row3
- U1 pad 20: row5 -> row2
- U1 pad 21: col2 -> row10
- U1 pad 22: col3 -> row9
- U1 pad 25: row9 -> row7
- U1 pad 26: row10 -> unconnected-(U1-Pad26)
- U1 pad 27: row11 -> unconnected-(U1-Pad27)
- U1 pad 30: Net-(SW_RESET1-Pad1) -> unconnected-(U1-Pad30)
- U1 pad 31: unconnected-(U1-Pad31) -> col2
- U1 pad 32: unconnected-(U1-Pad32) -> col3
- U1 pad 6: unconnected-(U1-Pad6) -> row0
- U1 pad 7: unconnected-(U1-Pad7) -> row1
- U1 pad 9: col0 -> unconnected-(U1-Pad9)
Routing:
- net col3: track 249.7 -> 529.2 mm
- net col2: track 245.7 -> 488.0 mm
- net col1: track 268.4 -> 504.6 mm
- net row11: track 27.6 -> 241.6 mm
- net row10: track 88.7 -> 274.8 mm
- net row9: track 81.7 -> 249.8 mm
- net row8: track 78.1 -> 231.1 mm
- net row7: track 52.9 -> 188.4 mm
- net row6: track 78.1 -> 195.9 mm
- net row0: track 21.6 -> 129.4 mm, vias 0 -> 1
- net row5: track 52.9 -> 148.0 mm
- net row1: track 25.1 -> 116.6 mm, vias 2 -> 4
- net row4: track 52.9 -> 125.9 mm
- net Net-(LED4-Pad2): track 0.00 -> 54.4 mm
- net row3: track 86.6 -> 137.8 mm
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- added copper zone on B.Cu, net GND
- added copper zone on F.Cu, net GND
Other:
- outline, holes or cut-outs redrawn

Commit message: :construction:
Parts:
- moved LED11 4.76 mm to (163.0, 194.0)
- moved LED12 4.76 mm to (115.4, 194.0)
- moved LED13 4.76 mm to (86.8, 165.4)
- moved LED8 4.76 mm to (305.9, 194.0)
- moved LED9 4.76 mm to (258.2, 194.0)
- moved LED6 4.76 mm to (334.4, 129.7)
- moved LED7 3.57 mm to (334.4, 166.6)
- moved LED1 1.19 mm to (86.8, 128.5)
Routing:
- net row2: track 83.2 -> 93.8 mm
- net Net-(LED6-Pad2): track 44.4 -> 34.6 mm
- net Net-(LED12-Pad2): track 45.0 -> 54.4 mm
- net row3: track 137.8 -> 129.4 mm
- net row4: track 125.9 -> 117.7 mm
- net Net-(LED5-Pad2): track 42.4 -> 50.1 mm
- net row5: track 148.0 -> 140.3 mm
- net row6: track 195.9 -> 189.1 mm
- net Net-(LED7-Pad2): track 47.8 -> 54.4 mm
- net VCC: track 670.8 -> 676.7 mm
- net Net-(LED10-Pad2): track 38.7 -> 43.3 mm
- net Net-(LED3-Pad2): track 75.8 -> 78.1 mm
- net Net-(LED10-Pad4): track 50.2 -> 52.0 mm
- net col3: track 529.2 -> 530.3 mm
- net Net-(LED8-Pad2): track 45.2 -> 44.1 mm
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Other:
- board size 277.7 x 90.2 mm -> 275.5 x 88.2 mm

Commit message: :construction:
Routing:
- net col2: track 488.7 -> 486.9 mm
- net col3: track 530.3 -> 528.7 mm
Other:
- outline, holes or cut-outs redrawn
