File: keyboard.kicad_pcb (KiCad board)
At the start: 2 copper layers, 275.5 x 88.2 mm, 100 parts, among them SW1 SW_PUSH, SW10 SW_PUSH, SW11 SW_PUSH, SW12 SW_PUSH, SW13 SW_PUSH, SW14 SW_PUSH, SW15 SW_PUSH, SW16 SW_PUSH, SW17 SW_PUSH, SW18 SW_PUSH, SW19 SW_PUSH, SW2 SW_PUSH, SW20 SW_PUSH, SW21 SW_PUSH, SW22 SW_PUSH, SW23 SW_PUSH, SW24 SW_PUSH, SW25 SW_PUSH, SW26 SW_PUSH, SW27 SW_PUSH, SW28 SW_PUSH, SW29 SW_PUSH, SW3 SW_PUSH, SW30 SW_PUSH, SW31 SW_PUSH, SW32 SW_PUSH, SW33 SW_PUSH, SW34 SW_PUSH, SW35 SW_PUSH, SW36 SW_PUSH, SW37 SW_PUSH, SW38 SW_PUSH, SW39 SW_PUSH, SW4 SW_PUSH, SW40 SW_PUSH, SW41 SW_PUSH, SW42 SW_PUSH, SW43 SW_PUSH, SW5 SW_PUSH, SW6 SW_PUSH, SW7 SW_PUSH, SW8 SW_PUSH, SW9 SW_PUSH, U1 Pico

Commit message: :sparkles: (all) before pcb order
Parts:
- moved D13 31.3 mm to (134.4, 153.4), turned to 180 degrees
- moved D14 13.9 mm to (142.7, 153.4), turned to 180 degrees
- moved Pico 1.10 mm to (100.9, 146.0)
- renumbered U1 to Pico
Routing:
- net row7: track 188.3 -> 293.1 mm
- net Net-(D13-Pad2): track 7.24 -> 43.5 mm
- net VCC: track 676.8 -> 656.6 mm
- net Net-(D14-Pad2): track 7.24 -> 24.1 mm
- net Net-(LED12-Pad2): track 54.4 -> 44.0 mm
- net row8: track 231.5 -> 226.0 mm
- net Net-(LED7-Pad2): track 54.4 -> 49.1 mm
- net row9: track 250.0 -> 245.2 mm
- net row10: track 275.5 -> 271.2 mm
- net Net-(LED5-Pad2): track 50.1 -> 47.6 mm
- net col1: track 504.6 -> 507.1 mm
- net Net-(LED1-Pad2): track 25.5 -> 23.1 mm
- net col2: track 486.9 -> 488.5 mm
- net Net-(D31-Pad2): track 7.24 -> 8.64 mm
- net col3: track 528.7 -> 530.0 mm
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
Commit message: :ambulance: (fix before order)
Other:
- board text added: "mechtech v1.0 PCB designed by kamo"
