File: keyboard.kicad_sch (KiCad schematic)
At the start: 88 parts, among them SW1 SW_PUSH, SW10 SW_PUSH, SW11 SW_PUSH, SW12 SW_PUSH, SW13 SW_PUSH, SW14 SW_PUSH, SW15 SW_PUSH, SW16 SW_PUSH, SW17 SW_PUSH, SW18 SW_PUSH, SW19 SW_PUSH, SW2 SW_PUSH, SW20 SW_PUSH, SW21 SW_PUSH, SW22 SW_PUSH, SW23 SW_PUSH, SW24 SW_PUSH, SW25 SW_PUSH, SW26 SW_PUSH, SW27 SW_PUSH, SW28 SW_PUSH, SW29 SW_PUSH, SW3 SW_PUSH, SW30 SW_PUSH, SW31 SW_PUSH, SW32 SW_PUSH, SW33 SW_PUSH, SW34 SW_PUSH, SW35 SW_PUSH, SW36 SW_PUSH, SW37 SW_PUSH, SW38 SW_PUSH, SW39 SW_PUSH, SW4 SW_PUSH, SW40 SW_PUSH, SW41 SW_PUSH, SW42 SW_PUSH, SW43 SW_PUSH, SW5 SW_PUSH, SW6 SW_PUSH, SW7 SW_PUSH, SW8 SW_PUSH, SW9 SW_PUSH, U1 Pico

Commit message: :sparkles: (pcb) in preparation
Parts:
- D1, D10, D11, D12, D13, D14, D15, D16, D17, D18, D19, D2, D20, D21, D22, D23, D24, D25, D26, D27, D28, D29, D3, D30, D31, D32, D33, D34, D35, D36, D37, D38, D39, D4, D40, D41, D42, D43, D5, D6, D7, D8, D9: footprint (none) -> kbd:D3_SMD_v2
- SW1, SW10, SW11, SW14, SW15, SW16, SW17, SW18, SW19, SW2, SW20, SW21, SW22, SW23, SW26, SW27, SW28, SW29, SW3, SW30, SW31, SW32, SW33, SW34, SW4, SW5, SW6, SW7, SW8, SW9: footprint (none) -> mikamo3:CherryMX_Hotswap_1u
- SW12: footprint (none) -> mikamo3:CherryMX_Hotswap_2u
- SW13, SW25: footprint (none) -> mikamo3:CherryMX_Hotswap_1.75u
- SW24, SW35, SW39: footprint (none) -> mikamo3:CherryMX_Hotswap_2.25u
- SW36, SW37, SW38, SW41, SW42, SW43: footprint (none) -> mikamo3:CherryMX_Hotswap_1.25u
- SW40: footprint (none) -> mikamo3:CherryMX_Hotswap_2.75u
- SW_RESET1: footprint (none) -> mikamo3:TactSwitch
- U1: footprint RPi_Pico:RPi_Pico_SMD_TH -> mikamo3:raspberry_pi_pico
Connections:
- net GND: no longer U1.42 (GND)
- no-connect marks 16 -> 17

Commit message: :construction:
Parts:
- D1, D10, D11, D12, D13, D14, D15, D16, D17, D18, D19, D2, D20, D21, D22, D23, D24, D25, D26, D27, D28, D29, D3, D30, D31, D32, D33, D34, D35, D36, D37, D38, D39, D4, D40, D41, D42, D43, D5, D6, D7, D8, D9: footprint kbd:D3_SMD_v2 -> Diode_SMD:D_SOD-123
- U1: symbol MCU_RaspberryPi_and_Boards:Pico -> mikamo3:Raspberry_Pi_Pico(without_debugPin)
Connections:
- net col2: now also U1.21 (GPIO16); no longer U1.11 (GPIO8)
- net col3: now also U1.22 (GPIO17); no longer U1.12 (GPIO9)
- net row6: now also U1.12 (GPIO9); no longer U1.21 (GPIO16)
- net row7: now also U1.11 (GPIO8); no longer U1.22 (GPIO17)
- no-connect marks 17 -> 14

Commit message: :construction:
Parts:
- added D44, D45, D46, D47, D48, D49: D, Diode_SMD:D_SOD-123, symbol Device:D
- added SW44, SW45, SW46, SW47: SW_PUSH, mikamo3:CherryMX_Hotswap_1u, symbol kbd:SW_PUSH
- added SW48, SW49: RotaryEncoder_Switch, Rotary_Encoder:RotaryEncoder_Alps_EC12E-Switch_Vertical_H20mm, symbol Device:RotaryEncoder_Switch
Connections:
- net GND: now also SW48.C, SW49.C
- net row0: now also SW44.1
- net row1: now also SW45.1
- net row2: now also SW46.1
- net row3: now also SW47.1
- net row4: now also SW48.S2
- net row5: now also SW49.S2
- net enc_0_a: now reaches U1.29 (GPIO22)
- net enc_0_a: now also SW48.A
- net enc_0_b: now reaches U1.31 (GPIO26_ADC0)
- net enc_0_b: now also SW48.B
- net enc_1_a: now reaches U1.32 (GPIO27_ADC1)
- net enc_1_a: now also SW49.A
- net enc_1_b: now reaches U1.34 (GPIO28_ADC2)
- net enc_1_b: now also SW49.B
- net col4: now reaches U1.7 (GPIO5)
- net col4: now also D44.1 (K), D45.1 (K), D46.1 (K), D47.1 (K), D48.1 (K), D49.1 (K)
- new net: D45.2 (A), SW45.2
- new net: D44.2 (A), SW44.2
- new net: D49.2 (A), SW49.S1
- new net: D46.2 (A), SW46.2
- new net: D47.2 (A), SW47.2
- new net: D48.2 (A), SW48.S1
- no-connect marks 14 -> 9
Other:
- moved on the sheet: D1, D10, D11, D12, D13, D14, D15, D16, D17, D18, D19, D2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

Commit message: :construction:
Parts:
- removed D44, D45, D46, D47, D48, D49: D, Diode_SMD:D_SOD-123, symbol Device:D
- removed SW44, SW45, SW46, SW47: SW_PUSH, mikamo3:CherryMX_Hotswap_1u, symbol kbd:SW_PUSH
- removed SW48, SW49: RotaryEncoder_Switch, Rotary_Encoder:RotaryEncoder_Alps_EC12E-Switch_Vertical_H20mm, symbol Device:RotaryEncoder_Switch
- added LED1, LED10, LED11, LED12, LED13, LED2, LED3, LED4, LED5, LED6, LED7, LED8, LED9: YS-SK6812MINI-E, mikamo3:YS-SK6812MINI-E, symbol kbd:YS-SK6812MINI-E
Connections:
- net GND: now also LED1.3 (VSS), LED10.3 (VSS), LED11.3 (VSS), LED12.3 (VSS), LED13.3 (VSS), LED2.3 (VSS), LED3.3 (VSS), LED4.3 (VSS), LED5.3 (VSS), LED6.3 (VSS), LED7.3 (VSS), LED8.3 (VSS), LED9.3 (VSS)
- net VCC: now also LED1.1 (VDD), LED10.1 (VDD), LED11.1 (VDD), LED12.1 (VDD), LED13.1 (VDD), LED2.1 (VDD), LED3.1 (VDD), LED4.1 (VDD), LED5.1 (VDD), LED6.1 (VDD), LED7.1 (VDD), LED8.1 (VDD), LED9.1 (VDD)
- net row10: now also SW43.1
- net row4: no longer SW40.1
- net row5: no longer SW41.1
- net row6: now also SW40.1; no longer SW42.1
- net row7: no longer SW43.1
- net row8: now also SW41.1
- net row9: now also SW42.1
- net led: now reaches U1.1 (GPIO0)
- net led: now also LED1.4 (DIN)
- net col4: no longer names the net of U1.7 (GPIO5)
- net enc_0_a: no longer names the net of U1.29 (GPIO22)
- net enc_0_b: no longer names the net of U1.31 (GPIO26_ADC0)
- net enc_1_a: no longer names the net of U1.32 (GPIO27_ADC1)
- net enc_1_b: no longer names the net of U1.34 (GPIO28_ADC2)
- new net: LED7.2 (DOUT), LED8.4 (DIN)
- new net: LED6.2 (DOUT), LED7.4 (DIN)
- new net: LED11.2 (DOUT), LED12.4 (DIN)
- new net: LED10.2 (DOUT), LED11.4 (DIN)
- new net: LED10.4 (DIN), LED9.2 (DOUT)
- new net: LED8.2 (DOUT), LED9.4 (DIN)
- new net: LED5.2 (DOUT), LED6.4 (DIN)
- new net: LED4.2 (DOUT), LED5.4 (DIN)
- new net: LED3.2 (DOUT), LED4.4 (DIN)
- new net: LED2.2 (DOUT), LED3.4 (DIN)
- new net: LED1.2 (DOUT), LED2.4 (DIN)
- new net: LED12.2 (DOUT), LED13.4 (DIN)
- no-connect marks 9 -> 14
Other:
- moved on the sheet: D40, D41, D42, D43, SW40, SW41, SW42, SW43

Commit message: :construction:
Parts:
- removed SW_RESET1: SW_Push, mikamo3:TactSwitch, symbol Switch:SW_Push
Connections:
- net col0: now also U1.11 (GPIO8); no longer U1.9 (GPIO6)
- net col1: now also U1.12 (GPIO9); no longer U1.10 (GPIO7)
- net col2: now also U1.31 (GPIO26_ADC0); no longer U1.21 (GPIO16)
- net col3: now also U1.32 (GPIO27_ADC1); no longer U1.22 (GPIO17)
- net row0: now also U1.6 (GPIO4); no longer U1.14 (GPIO10)
- net row1: now also U1.7 (GPIO5); no longer U1.15 (GPIO11)
- net row10: now also U1.21 (GPIO16); no longer U1.26 (GPIO20)
- net row11: now also U1.14 (GPIO10); no longer U1.27 (GPIO21)
- net row2: now also U1.20 (GPIO15); no longer U1.16 (GPIO12)
- net row3: now also U1.19 (GPIO14); no longer U1.17 (GPIO13)
- net row4: now also U1.17 (GPIO13); no longer U1.19 (GPIO14)
- net row5: now also U1.16 (GPIO12); no longer U1.20 (GPIO15)
- net row6: now also U1.15 (GPIO11); no longer U1.12 (GPIO9)
- net row7: now also U1.25 (GPIO19); no longer U1.11 (GPIO8)
- net row9: now also U1.22 (GPIO17); no longer U1.25 (GPIO19)
- no-connect marks 14 -> 13

Commit message: :sparkles: (all) before pcb order
Parts:
- renumbered U1 to Pico
Changed lines of the file:
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@@
   (symbol (lib_id "mikamo3:Raspberry_Pi_Pico(without_debugPin)") (at 43.18 49.53 0) (unit 1)
     (in_bom yes) (on_board yes) (fields_autoplaced)
-    (property "Reference" "U1" (id 0) (at 43.18 17.78 0))
+    (property "Reference" "Pico" (id 0) (at 43.18 17.78 0))
     (property "Value" "Pico" (id 1) (at 43.18 20.32 0))
     (property "Footprint" "mikamo3:raspberry_pi_pico" (id 2) (at 43.18 49.53 90)
@@
       (reference "LED13") (unit 1) (value "YS-SK6812MINI-E") (footprint "mikamo3:YS-SK6812MINI-E")
     )
+    (path "/d62990f7-f6d3-4d28-a6c5-3edf4b260501"
+      (reference "Pico") (unit 1) (value "Pico") (footprint "mikamo3:raspberry_pi_pico")
+    )
     (path "/a4f1aa9d-559e-4977-b38d-408ec59e07b2"
       (reference "SW1") (unit 1) (value "SW_PUSH") (footprint "mikamo3:CherryMX_Hotswap_1u")
@@
       (reference "SW43") (unit 1) (value "SW_PUSH") (footprint "mikamo3:CherryMX_Hotswap_1.25u")
     )
-    (path "/d62990f7-f6d3-4d28-a6c5-3edf4b260501"
-      (reference "U1") (unit 1) (value "Pico") (footprint "mikamo3:raspberry_pi_pico")
-    )
-  )
+  )
